File: MotorDriverV2/_autosave-uController_sch.kicad_sch (KiCad schematic)
At the start: 1 part, among them IC3 ESP32-S2FH4

Commit message: UPDATE: Added symbols, fotprints and datasheets for components
Parts:
- removed IC3: ESP32-S2FH4, QFN40P700X700X90-57N-D, symbol ESP32-S2FH4:ESP32-S2FH4
Changed lines of the file:
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@@
 	(generator_version "9.0")
 	(paper "A4")
-	(symbol
-		(lib_id "ESP32-S2FH4:ESP32-S2FH4")
-		(at 96.52 92.71 0)
-		(unit 1)
-		(exclude_from_sim no)
-		(in_bom yes)
-		(on_board yes)
-		(dnp no)
-		(fields_autoplaced yes)
-		(property "Reference" "IC3"
-			(at 151.13 86.2898 0)
-			(effects
-				(font
-					(size 1.27 1.27)
-				)
-			)
-		)
-		(property "Value" "ESP32-S2FH4"
-			(at 151.13 88.8298 0)
-			(effects
-				(font
-					(size 1.27 1.27)
-				)
-			)
-		)
-		(property "Footprint" "QFN40P700X700X90-57N-D"
-			(at 143.51 172.39 0)
-			(effects
-				(font
-					(size 1.27 1.27)
-				)
-				(justify left top)
-				(hide yes)
-			)
-		)
-		(property "Datasheet" ""
-			(at 143.51 272.39 0)
-			(effects
-				(font
-					(size 1.27 1.27)
-				)
-				(justify left top)
-				(hide yes)
-			)
-		)
-		(property "Description" "ESP32-S2FH4"
-			(at 96.52 92.71 0)
-			(effects
-				(font
-					(size 1.27 1.27)
-				)
-				(hide yes)
-			)
-		)
-		(property "Height" "0.9"
-			(at 143.51 472.39 0)
-			(effects
-				(font
-					(size 1.27 1.27)
-				)
-				(justify left top)
-				(hide yes)
-			)
-		)
-		(property "Mouser Part Number" "356-ESP32-S2FH4"
-			(at 143.51 572.39 0)
-			(effects
-				(font
-					(size 1.27 1.27)
-				)
-				(justify left top)
-				(hide yes)
-			)
-		)
-		(property "Mouser Price/Stock" "https://www.mouser.co.uk/ProductDetail/Espressif-Systems/ESP32-S2FH4?qs=DPoM0jnrROVef2vYCoSa1w%3D%3D"
-			(at 143.51 672.39 0)
-			(effects
-				(font
-					(size 1.27 1.27)
-				)
-				(justify left top)
-				(hide yes)
-			)
-		)
-		(property "Manufacturer_Name" "Espressif Systems"
-			(at 143.51 772.39 0)
-			(effects
-				(font
-					(size 1.27 1.27)
-				)
-				(justify left top)
-				(hide yes)
-			)
-		)
-		(property "Manufacturer_Part_Number" "ESP32-S2FH4"
-			(at 143.51 872.39 0)
-			(effects
-				(font
-					(size 1.27 1.27)
-				)
-				(justify left top)
-				(hide yes)
-			)
-		)
-		(pin "1"
-		)
-		(pin "4"
-		)
-		(pin "9"
-		)
-		(pin "8"
-		)
-		(pin "3"
-		)
-		(pin "11"
-		)
-		(pin "56"
-		)
-		(pin "7"
-		)
-		(pin "14"
-		)
-		(pin "2"
-		)
-		(pin "5"
-		)
-		(pin "6"
-		)
-		(pin "10"
-		)
-		(pin "12"
-		)
-		(pin "13"
-		)
-		(pin "57"
-		)
-		(pin "15"
-		)
-		(pin "17"
-		)
-		(pin "46"
-		)
-		(pin "55"
-		)
-		(pin "18"
-		)
-		(pin "23"
-		)
-		(pin "19"
-		)
-		(pin "44"
-		)
-		(pin "53"
-		)
-		(pin "45"
-		)
-		(pin "52"
-		)
-		(pin "50"
-		)
-		(pin "20"
-		)
-		(pin "21"
-		)
-		(pin "51"
-		)
-		(pin "22"
-		)
-		(pin "16"
-		)
-		(pin "49"
-		)
-		(pin "48"
-		)
-		(pin "54"
-		)
-		(pin "24"
-		)
-		(pin "47"
-		)
-		(pin "25"
-		)
-		(pin "26"
-		)
-		(pin "27"
-		)
-		(pin "43"
-		)
-		(pin "41"
-		)
-		(pin "42"
-		)
-		(pin "29"
-		)
-		(pin "37"
-		)
-		(pin "39"
-		)
-		(pin "34"
-		)
-		(pin "36"
-		)
-		(pin "33"
-		)
-		(pin "38"
-		)
-		(pin "32"
-		)
-		(pin "31"
-		)
-		(pin "30"
-		)
-		(pin "40"
-		)
-		(pin "28"
-		)
-		(pin "35"
-		)
-		(instances
-			(project ""
-				(path "/9a6a3a05-adb1-47eb-a38b-9a704717c7ef/99db9728-3194-4b24-aa4b-533760f9cc37"
-					(reference "IC3")
-					(unit 1)
-				)
-			)
-		)
-	)
 )
