File: MotorDriverV2/MotorDriver.kicad_sch (KiCad schematic)
At the start: 12 parts, among them IC1 DRV8871DDARQ1, IC2 DRV8871DDARQ1, J2 Out_A, J3 Out_A, J4 Out_B, J5 Out_B

Commit message: UPDATE: Schematic
Parts:
- removed J2: Out_A, Connector_JST:JST_XH_B2B-XH-A_1x02_P2.50mm_Vertical, symbol Connector:Conn_01x02_Pin
- removed J4: Out_B, Connector_JST:JST_XH_B2B-XH-A_1x02_P2.50mm_Vertical, symbol Connector:Conn_01x02_Pin
