File: MotorDriverV2/uController.kicad_sch (KiCad schematic)
At the start: 0 parts

Commit message: UPDATE: Schematic
Parts:
- added C5: 100uF, symbol Device:C
- added C6: 100nF, symbol Device:C
- added C8: 10uF, symbol Device:C
- added D1: LED, symbol Device:LED
- added IC3: ESP32-S3-WROOM-1U-N4, ESP32-S3-WROOM-1U-N4:ESP32S3WROOM1UN4, symbol ESP32-S3-WROOM-1U-N4:ESP32-S3-WROOM-1U-N4
- added J2: USB_C_Receptacle_USB2.0_14P, symbol Connector:USB_C_Receptacle_USB2.0_14P
- added PS1: LM1117IMPX-3.3_NOPB, SOT230P700X180-4N, symbol LM1117IMPX-3_3_NOPB:LM1117IMPX-3.3_NOPB
- added R3, R4: 5k1, symbol Device:R
- added R5: 100, symbol Device:R
- added S1, S2: PTS636SKG25JSMTR_LFS, PTS636SKG25JSMTR_LFS:PTS636SKG25JSMTRLFS, symbol PTS636SKG25JSMTR_LFS:PTS636SKG25JSMTR_LFS
- added U1: USBLC6-2SC6, Package_TO_SOT_SMD:SOT-23-6, symbol Power_Protection:USBLC6-2SC6
Connections:
- new net: J2.A7 (D-), J2.B7 (D-), U1.1 (I/O1)
- new net: J2.A6 (D+), J2.B6 (D+), U1.3 (I/O2)
- new net: D1.2 (A), R5.2
- new net: J2.A5 (CC1), R3.1
- new net: J2.B5 (CC2), R4.1
- new net +3V3: C5.1, C6.1, PS1.2 (OUTPUT), PS1.4 (VOUT), R5.1
- new net +5V: C8.1, PS1.3 (INPUT)
- new net D+: U1.4 (I/O2)
- new net D-: U1.6 (I/O1)
- new net GND: C5.2, C6.2, C8.2, D1.1 (K), IC3.1 (GND_1), IC3.40 (GND_2), IC3.41 (GND_3), IC3.42 (GND_4), IC3.43 (GND_5), IC3.44 (GND_6), IC3.45 (GND_7), IC3.46 (GND_8), IC3.47 (GND_9), IC3.48 (GND_10), IC3.49 (GND_11), J2.A1 (GND), J2.A12 (GND), J2.B1 (GND), J2.B12 (GND), J2.S1 (SHIELD), PS1.1 (ADJ/GND), R3.2, R4.2, S1.3 (GND_1), S1.4 (GND_2), S2.3 (GND_1), S2.4 (GND_2), U1.2 (GND)
- new net In1_1: IC3.7 (IO7)
- new net In1_2: IC3.6 (IO6)
- new net In2_1: IC3.4 (IO4)
- new net In2_2: IC3.5 (IO5)
- new net VBUS: J2.A4 (VBUS), J2.A9 (VBUS), J2.B4 (VBUS), J2.B9 (VBUS), U1.5 (VBUS)
- new net boot: IC3.27 (IO0)
- no-connect marks 0 -> 31
